File: PCB/F18_DDI.kicad_sch (KiCad schematic)
At the start: 47 parts

Commit message: Finish electrical schematic
Parts:
- added R12, R13, R14, R15, R20, R21, R22, R23, R28, R29, R30, R31, R36, R37, R38, R39, R4, R5, R6, R7: 10K, Resistor_SMD:R_0805_2012Metric, symbol Device:R_Small
- R1, R2, R3: footprint (none) -> Resistor_SMD:R_0805_2012Metric
- R10: renamed from R6; footprint (none) -> Resistor_SMD:R_0805_2012Metric
- R11: renamed from R7; footprint (none) -> Resistor_SMD:R_0805_2012Metric
- R16: renamed from R8; footprint (none) -> Resistor_SMD:R_0805_2012Metric
- R17: renamed from R9; footprint (none) -> Resistor_SMD:R_0805_2012Metric
- R18: renamed from R10; footprint (none) -> Resistor_SMD:R_0805_2012Metric
- R19: renamed from R11; footprint (none) -> Resistor_SMD:R_0805_2012Metric
- R24: renamed from R12; footprint (none) -> Resistor_SMD:R_0805_2012Metric
- R25: renamed from R13; footprint (none) -> Resistor_SMD:R_0805_2012Metric
- R26: renamed from R14; footprint (none) -> Resistor_SMD:R_0805_2012Metric
- R27: renamed from R15; footprint (none) -> Resistor_SMD:R_0805_2012Metric
- R32: renamed from R16; footprint (none) -> Resistor_SMD:R_0805_2012Metric
- R33: renamed from R17; footprint (none) -> Resistor_SMD:R_0805_2012Metric
- R34: renamed from R18; footprint (none) -> Resistor_SMD:R_0805_2012Metric
- R35: renamed from R19; footprint (none) -> Resistor_SMD:R_0805_2012Metric
- R40: renamed from R20; footprint (none) -> Resistor_SMD:R_0805_2012Metric
- R41: renamed from R21; footprint (none) -> Resistor_SMD:R_0805_2012Metric
- R42: renamed from R22; footprint (none) -> Resistor_SMD:R_0805_2012Metric
- R43: renamed from R23; footprint (none) -> Resistor_SMD:R_0805_2012Metric
- R8: renamed from R4; footprint (none) -> Resistor_SMD:R_0805_2012Metric
- R9: renamed from R5; footprint (none) -> Resistor_SMD:R_0805_2012Metric
- renumbered S21 to S1, S3 to S10, S8 to S11, S13 to S12, S18 to S13, S4 to S14, S9 to S15, S14 to S16, S19 to S17, S5 to S18, S10 to S19, S1 to S2, S15 to S20, S20 to S21, S6 to S3, S11 to S4, S16 to S5, S2 to S6, S12 to S8, S17 to S9
Connections:
- net +3.3V: now also S10.3, S10.4, S11.3, S11.4, S12.3, S12.4, S13.3, S13.4, S14.3, S14.4, S15.3, S15.4, S16.3, S16.4, S17.3, S17.4, S18.3, S18.4, S19.3, S19.4, S20.3, S20.4, S21.3, S21.4, S6.3, S6.4, S7.3, S7.4, S8.3, S8.4, S9.3, S9.4
- net GND: now also R12.1, R13.1, R14.1, R15.1, R20.1, R21.1, R22.1, R23.1, R28.1, R29.1, R30.1, R31.1, R36.1, R37.1, R38.1, R39.1, R4.1, R5.1, R6.1, R7.1
- net Switch Pos 1: now also A1.26 (GPIO20); no longer A1.1 (GPIO0)
- net Switch Pos 2: now also A1.27 (GPIO21); no longer A1.2 (GPIO1)
- net Switch Pos 3: now also A1.29 (GPIO22); no longer A1.4 (GPIO2)
- net Button10: now reaches S19.1
- net Button10: now also A1.12 (GPIO9), S19.2, R37.2
- net Button8: now reaches S11.1
- net Button8: now also A1.10 (GPIO7), S11.2, R21.2
- net Button9: now reaches S15.1
- net Button9: now also A1.11 (GPIO8), S15.2, R29.2
- net Button4: now reaches S14.1
- net Button4: now also A1.5 (GPIO3), S14.2, R28.2
- net Button6: now reaches S3.1
- net Button6: now also A1.7 (GPIO5), S3.2, R5.2
- net Button13: now reaches S12.1
- net Button13: now also A1.16 (GPIO12), S12.2, R22.2
- net Button7: now reaches S7.1
- net Button7: now also A1.9 (GPIO6), S7.2, R13.2
- net Button15: now reaches S20.1
- net Button15: now also A1.19 (GPIO14), S20.2, R38.2
- net Button11: now reaches A1.14 (GPIO10)
- net Button11: now also S4.1, S4.2, R6.2
- net Button12: now reaches A1.15 (GPIO11)
- net Button12: now also S8.1, S8.2, R14.2
- net Button14: now reaches A1.17 (GPIO13)
- net Button14: now also S16.1, S16.2, R30.2
- net Button16: now reaches A1.20 (GPIO15)
- net Button16: now also S5.1, S5.2, R7.2
- net Button17: now reaches A1.21 (GPIO16)
- net Button17: now also S9.1, S9.2, R15.2
- net Button18: now reaches A1.22 (GPIO17)
- net Button18: now also S13.1, S13.2, R23.2
- net Button19: now reaches A1.24 (GPIO18)
- net Button19: now also S17.1, S17.2, R31.2
- net Button20: now reaches A1.25 (GPIO19)
- net Button20: now also S21.1, S21.2, R39.2
- net Button5: now reaches A1.6 (GPIO4)
- net Button5: now also S18.1, S18.2, R36.2
- net Button3: now reaches S10.1
- net Button3: now also A1.4 (GPIO2), S10.2, R20.2
- net Button1: now reaches S2.1
- net Button1: now also A1.1 (GPIO0), S2.2, R4.2
- net Button2: now reaches S6.1
- net Button2: now also A1.2 (GPIO1), S6.2, R12.2
- no-connect marks 0 -> 5

Commit message: preliminary pcb layout
Parts:
- R1, R10, R11, R12, R13, R14, R15, R16, R17, R18, R19, R2, R20, R21, R22, R23, R24, R25, R26, R27, R28, R29, R3, R30, R31, R32, R33, R34, R35, R36, R37, R38, R39, R4, R40, R41, R42, R43, R5, R6, R7, R8, R9: footprint Resistor_SMD:R_0805_2012Metric -> Resistor_SMD:R_1206_3216Metric_Pad1.30x1.75mm_HandSolder
Changed lines of the file:
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@@
 			)
 		)
-		(property "Footprint" "Resistor_SMD:R_0805_2012Metric"
+		(property "Footprint" "Resistor_SMD:R_1206_3216Metric_Pad1.30x1.75mm_HandSolder"
 			(at 347.98 201.93 0)
 			(effects
@@
 			)
 		)
-		(property "Footprint" "Resistor_SMD:R_0805_2012Metric"
+		(property "Footprint" "Resistor_SMD:R_1206_3216Metric_Pad1.30x1.75mm_HandSolder"
 			(at 215.9 95.25 0)
 			(effects
@@
 			)
 		)
-		(property "Footprint" "Resistor_SMD:R_0805_2012Metric"
+		(property "Footprint" "Resistor_SMD:R_1206_3216Metric_Pad1.30x1.75mm_HandSolder"
 			(at 375.92 219.71 0)
 			(effects
@@
 			)
 		)
-		(property "Footprint" "Resistor_SMD:R_0805_2012Metric"
+		(property "Footprint" "Resistor_SMD:R_1206_3216Metric_Pad1.30x1.75mm_HandSolder"
 			(at 215.9 201.93 0)
 			(effects
@@
 			)
 		)
-		(property "Footprint" "Resistor_SMD:R_0805_2012Metric"
+		(property "Footprint" "Resistor_SMD:R_1206_3216Metric_Pad1.30x1.75mm_HandSolder"
 			(at 242.57 163.83 0)
 			(effects
@@
 			)
 		)
-		(property "Footprint" "Resistor_SMD:R_0805_2012Metric"
+		(property "Footprint" "Resistor_SMD:R_1206_3216Metric_Pad1.30x1.75mm_HandSolder"
 			(at 375.92 113.03 0)
 			(effects
@@
 			)
 		)
-		(property "Footprint" "Resistor_SMD:R_0805_2012Metric"
+		(property "Footprint" "Resistor_SMD:R_1206_3216Metric_Pad1.30x1.75mm_HandSolder"
 			(at 330.2 219.71 0)
 			(effects
@@
 			)
 		)
-		(property "Footprint" "Resistor_SMD:R_0805_2012Metric"
+		(property "Footprint" "Resistor_SMD:R_1206_3216Metric_Pad1.30x1.75mm_HandSolder"
 			(at 198.12 67.31 0)
 			(effects
@@
 			)
 		)
-		(property "Footprint" "Resistor_SMD:R_0805_2012Metric"
+		(property "Footprint" "Resistor_SMD:R_1206_3216Metric_Pad1.30x1.75mm_HandSolder"
 			(at 33.02 147.32 0)
 			(effects
@@
 			)
 		)
-		(property "Footprint" "Resistor_SMD:R_0805_2012Metric"
+		(property "Footprint" "Resistor_SMD:R_1206_3216Metric_Pad1.30x1.75mm_HandSolder"
 			(at 242.57 113.03 0)
 			(effects
@@
 			)
 		)
-		(property "Footprint" "Resistor_SMD:R_0805_2012Metric"
+		(property "Footprint" "Resistor_SMD:R_1206_3216Metric_Pad1.30x1.75mm_HandSolder"
 			(at 304.8 49.53 0)
 			(effects
@@
 			)
 		)
-		(property "Footprint" "Resistor_SMD:R_0805_2012Metric"
+		(property "Footprint" "Resistor_SMD:R_1206_3216Metric_Pad1.30x1.75mm_HandSolder"
 			(at 242.57 219.71 0)
 			(effects
@@
 			)
 		)
-		(property "Footprint" "Resistor_SMD:R_0805_2012Metric"
+		(property "Footprint" "Resistor_SMD:R_1206_3216Metric_Pad1.30x1.75mm_HandSolder"
 			(at 260.35 201.93 0)
 			(effects
@@
 			)
 		)
-		(property "Footprint" "Resistor_SMD:R_0805_2012Metric"
+		(property "Footprint" "Resistor_SMD:R_1206_3216Metric_Pad1.30x1.75mm_HandSolder"
 			(at 330.2 113.03 0)
 			(effects
@@
 			)
 		)
-		(property "Footprint" "Resistor_SMD:R_0805_2012Metric"
+		(property "Footprint" "Resistor_SMD:R_1206_3216Metric_Pad1.30x1.75mm_HandSolder"
 			(at 242.57 67.31 0)
 			(effects
@@
 			)
 		)
-		(property "Footprint" "Resistor_SMD:R_0805_2012Metric"
+		(property "Footprint" "Resistor_SMD:R_1206_3216Metric_Pad1.30x1.75mm_HandSolder"
 			(at 215.9 146.05 0)
 			(effects
@@
 			)
 		)
-		(property "Footprint" "Resistor_SMD:R_0805_2012Metric"
+		(property "Footprint" "Resistor_SMD:R_1206_3216Metric_Pad1.30x1.75mm_HandSolder"
 			(at 393.7 146.05 0)
 			(effects
@@
 			)
 		)
-		(property "Footprint" "Resistor_SMD:R_0805_2012Metric"
+		(property "Footprint" "Resistor_SMD:R_1206_3216Metric_Pad1.30x1.75mm_HandSolder"
 			(at 347.98 95.25 0)
 			(effects
@@
 			)
 		)
-		(property "Footprint" "Resistor_SMD:R_0805_2012Metric"
+		(property "Footprint" "Resistor_SMD:R_1206_3216Metric_Pad1.30x1.75mm_HandSolder"
 			(at 304.8 146.05 0)
 			(effects
@@
 			)
 		)
-		(property "Footprint" "Resistor_SMD:R_0805_2012Metric"
+		(property "Footprint" "Resistor_SMD:R_1206_3216Metric_Pad1.30x1.75mm_HandSolder"
 			(at 35.56 153.67 0)
 			(effects
@@
 			)
 		)
-		(property "Footprint" "Resistor_SMD:R_0805_2012Metric"
+		(property "Footprint" "Resistor_SMD:R_1206_3216Metric_Pad1.30x1.75mm_HandSolder"
 			(at 393.7 49.53 0)
 			(effects
@@
 			)
 		)
-		(property "Footprint" "Resistor_SMD:R_0805_2012Metric"
+		(property "Footprint" "Resistor_SMD:R_1206_3216Metric_Pad1.30x1.75mm_HandSolder"
 			(at 393.7 95.25 0)
 			(effects
@@
 			)
 		)
-		(property "Footprint" "Resistor_SMD:R_0805_2012Metric"
+		(property "Footprint" "Resistor_SMD:R_1206_3216Metric_Pad1.30x1.75mm_HandSolder"
 			(at 330.2 163.83 0)
 			(effects
@@
 			)
 		)
-		(property "Footprint" "Resistor_SMD:R_0805_2012Metric"
+		(property "Footprint" "Resistor_SMD:R_1206_3216Metric_Pad1.30x1.75mm_HandSolder"
 			(at 215.9 49.53 0)
 			(effects
@@
 			)
 		)
-		(property "Footprint" "Resistor_SMD:R_0805_2012Metric"
+		(property "Footprint" "Resistor_SMD:R_1206_3216Metric_Pad1.30x1.75mm_HandSolder"
 			(at 330.2 67.31 0)
 			(effects
@@
 			)
 		)
-		(property "Footprint" "Resistor_SMD:R_0805_2012Metric"
+		(property "Footprint" "Resistor_SMD:R_1206_3216Metric_Pad1.30x1.75mm_HandSolder"
 			(at 287.02 219.71 0)
 			(effects
@@
 			)
 		)
-		(property "Footprint" "Resistor_SMD:R_0805_2012Metric"
+		(property "Footprint" "Resistor_SMD:R_1206_3216Metric_Pad1.30x1.75mm_HandSolder"
 			(at 304.8 201.93 0)
 			(effects
@@
 			)
 		)
-		(property "Footprint" "Resistor_SMD:R_0805_2012Metric"
+		(property "Footprint" "Resistor_SMD:R_1206_3216Metric_Pad1.30x1.75mm_HandSolder"
 			(at 198.12 163.83 0)
 			(effects
@@
 			)
 		)
-		(property "Footprint" "Resistor_SMD:R_0805_2012Metric"
+		(property "Footprint" "Resistor_SMD:R_1206_3216Metric_Pad1.30x1.75mm_HandSolder"
 			(at 375.92 67.31 0)
 			(effects
@@
 			)
 		)
-		(property "Footprint" "Resistor_SMD:R_0805_2012Metric"
+		(property "Footprint" "Resistor_SMD:R_1206_3216Metric_Pad1.30x1.75mm_HandSolder"
 			(at 393.7 201.93 0)
 			(effects
@@
 			)
 		)
-		(property "Footprint" "Resistor_SMD:R_0805_2012Metric"
+		(property "Footprint" "Resistor_SMD:R_1206_3216Metric_Pad1.30x1.75mm_HandSolder"
 			(at 287.02 163.83 0)
 			(effects
@@
 			)
 		)
-		(property "Footprint" "Resistor_SMD:R_0805_2012Metric"
+		(property "Footprint" "Resistor_SMD:R_1206_3216Metric_Pad1.30x1.75mm_HandSolder"
 			(at 260.35 95.25 0)
 			(effects
@@
 			)
 		)
-		(property "Footprint" "Resistor_SMD:R_0805_2012Metric"
+		(property "Footprint" "Resistor_SMD:R_1206_3216Metric_Pad1.30x1.75mm_HandSolder"
 			(at 260.35 49.53 0)
 			(effects
@@
 			)
 		)
-		(property "Footprint" "Resistor_SMD:R_0805_2012Metric"
+		(property "Footprint" "Resistor_SMD:R_1206_3216Metric_Pad1.30x1.75mm_HandSolder"
 			(at 304.8 95.25 0)
 			(effects
@@
 			)
 		)
-		(property "Footprint" "Resistor_SMD:R_0805_2012Metric"
+		(property "Footprint" "Resistor_SMD:R_1206_3216Metric_Pad1.30x1.75mm_HandSolder"
 			(at 260.35 146.05 0)
 			(effects
@@
 			)
 		)
-		(property "Footprint" "Resistor_SMD:R_0805_2012Metric"
+		(property "Footprint" "Resistor_SMD:R_1206_3216Metric_Pad1.30x1.75mm_HandSolder"
 			(at 347.98 146.05 0)
 			(effects
@@
 			)
 		)
-		(property "Footprint" "Resistor_SMD:R_0805_2012Metric"
+		(property "Footprint" "Resistor_SMD:R_1206_3216Metric_Pad1.30x1.75mm_HandSolder"
 			(at 287.02 67.31 0)
 			(effects
@@
 			)
 		)
-		(property "Footprint" "Resistor_SMD:R_0805_2012Metric"
+		(property "Footprint" "Resistor_SMD:R_1206_3216Metric_Pad1.30x1.75mm_HandSolder"
 			(at 198.12 113.03 0)
 			(effects
@@
 			)
 		)
-		(property "Footprint" "Resistor_SMD:R_0805_2012Metric"
+		(property "Footprint" "Resistor_SMD:R_1206_3216Metric_Pad1.30x1.75mm_HandSolder"
 			(at 287.02 113.03 0)
 			(effects
@@
 			)
 		)
-		(property "Footprint" "Resistor_SMD:R_0805_2012Metric"
+		(property "Footprint" "Resistor_SMD:R_1206_3216Metric_Pad1.30x1.75mm_HandSolder"
 			(at 198.12 219.71 0)
 			(effects
@@
 			)
 		)
-		(property "Footprint" "Resistor_SMD:R_0805_2012Metric"
+		(property "Footprint" "Resistor_SMD:R_1206_3216Metric_Pad1.30x1.75mm_HandSolder"
 			(at 30.48 140.97 0)
 			(effects
@@
 			)
 		)
-		(property "Footprint" "Resistor_SMD:R_0805_2012Metric"
+		(property "Footprint" "Resistor_SMD:R_1206_3216Metric_Pad1.30x1.75mm_HandSolder"
 			(at 347.98 49.53 0)
 			(effects
@@
 			)
 		)
-		(property "Footprint" "Resistor_SMD:R_0805_2012Metric"
+		(property "Footprint" "Resistor_SMD:R_1206_3216Metric_Pad1.30x1.75mm_HandSolder"
 			(at 375.92 163.83 0)
 			(effects

Commit message: Finalize PCB
Parts:
- added H1, H2: MountingHole_Pad, MountingHole:MountingHole_3.2mm_M3_DIN965_Pad, symbol Mechanical:MountingHole_Pad
Connections:
- net Button1: now also A1.20 (GPIO15); no longer A1.1 (GPIO0)
- net Button10: now also A1.10 (GPIO7); no longer A1.12 (GPIO9)
- net Button11: now also A1.26 (GPIO20); no longer A1.14 (GPIO10)
- net Button12: now also A1.17 (GPIO13); no longer A1.15 (GPIO11)
- net Button13: now also A1.6 (GPIO4); no longer A1.16 (GPIO12)
- net Button14: now also A1.1 (GPIO0); no longer A1.17 (GPIO13)
- net Button15: now also A1.12 (GPIO9); no longer A1.19 (GPIO14)
- net Button16: now also A1.27 (GPIO21); no longer A1.20 (GPIO15)
- net Button17: now also A1.16 (GPIO12); no longer A1.21 (GPIO16)
- net Button18: now also A1.5 (GPIO3); no longer A1.22 (GPIO17)
- net Button19: now also A1.7 (GPIO5); no longer A1.24 (GPIO18)
- net Button2: now also A1.29 (GPIO22); no longer A1.2 (GPIO1)
- net Button20: now also A1.11 (GPIO8); no longer A1.25 (GPIO19)
- net Button3: now also A1.15 (GPIO11); no longer A1.4 (GPIO2)
- net Button4: now also A1.4 (GPIO2); no longer A1.5 (GPIO3)
- net Button5: now also A1.9 (GPIO6); no longer A1.6 (GPIO4)
- net Button6: now also A1.25 (GPIO19); no longer A1.7 (GPIO5)
- net Button7: now also A1.19 (GPIO14); no longer A1.9 (GPIO6)
- net Button8: now also A1.14 (GPIO10); no longer A1.10 (GPIO7)
- net Button9: now also A1.2 (GPIO1); no longer A1.11 (GPIO8)
- net GND: now also H1.1, H2.1
- net Switch Pos 1: now also A1.21 (GPIO16); no longer A1.26 (GPIO20)
- net Switch Pos 2: now also A1.22 (GPIO17); no longer A1.27 (GPIO21)
- net Switch Pos 3: now also A1.24 (GPIO18); no longer A1.29 (GPIO22)
