File: PCB/F18_DDI.kicad_pcb (KiCad board)
At the start: 2 copper layers, 196.1 x 194.1 mm, 67 parts

Commit message: preliminary pcb layout
Parts:
- A1: moved to B.Cu
- R1, R10, R11, R12, R13, R14, R15, R16, R17, R18, R19, R2, R20, R21, R22, R23, R24, R25, R26, R27, R28, R29, R3, R30, R31, R32, R33, R34, R35, R36, R37, R38, R39, R4, R40, R41, R42, R43, R5, R6, R7, R8, R9: footprint Resistor_SMD:R_0805_2012Metric -> Resistor_SMD:R_1206_3216Metric_Pad1.30x1.75mm_HandSolder; moved to B.Cu
- moved R39 211.2 mm to (248.5, 241.5), turned to 180 degrees
- moved R43 209.7 mm to (249.5, 251.0)
- moved A1 207.4 mm to (254.1, 80.8), turned to 90 degrees
- moved VR2 206.6 mm to (268.8, 250.0)
- moved S16 206.1 mm to (273.5, 211.8)
- moved R38 204.3 mm to (228.4, 241.5), turned to 180 degrees
- moved S15 203.0 mm to (273.5, 191.8)
- moved R42 202.8 mm to (228.6, 251.5)
- moved S14 202.4 mm to (273.5, 171.8)
- moved R37 198.9 mm to (208.4, 241.0), turned to 180 degrees
- moved R41 197.7 mm to (208.6, 251.5)
- moved R30 196.4 mm to (267.0, 206.6), turned to -90 degrees
- moved R40 194.7 mm to (189.0, 251.5)
- moved R34 193.7 mm to (275.5, 206.4), turned to 90 degrees
- moved S21 189.9 mm to (242.2, 243.1)
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Routing:
- net +5V: track 0.00 -> 758.3 mm
- net Potentiometer 1: track 0.00 -> 293.3 mm
- net /Button19: track 0.00 -> 275.4 mm
- net /Button5: track 0.00 -> 256.2 mm
- net /Button2: track 0.00 -> 251.4 mm
- net /Button10: track 0.00 -> 229.2 mm
- net Potentiometer 2: track 0.00 -> 229.1 mm
- net /Button16: track 0.00 -> 217.4 mm
- net /Button11: track 0.00 -> 213.3 mm
- net /Button15: track 0.00 -> 209.5 mm
- net /Button6: track 0.00 -> 197.7 mm
- net /Button20: track 0.00 -> 186.7 mm
- net /Button1: track 0.00 -> 146.4 mm
- net /Button14: track 0.00 -> 146.0 mm
- net /Button9: track 0.00 -> 124.5 mm
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- added copper zone on F.Cu, net +3.3V
- added copper zone on B.Cu, net GND
Other:
- board size 196.1 x 194.1 mm -> 160.2 x 190.1 mm

Commit message: Finalize PCB
Parts:
- added H1: MountingHole_Pad, MountingHole:MountingHole_3.2mm_M3_DIN965_Pad, F.Cu at (130.0, 75.0)
- added H2: MountingHole_Pad, MountingHole:MountingHole_3.2mm_M3_DIN965_Pad, F.Cu at (145.0, 246.2)
- moved R43 3.87 mm to (248.6, 247.2)
- moved R3 2.50 mm to (192.0, 81.0)
- moved S1 2.22 mm to (201.4, 90.8)
- moved R14 2.06 mm to (189.1, 100.5)
- moved R15 2.06 mm to (209.4, 100.5)
- moved R21 2.00 mm to (249.1, 100.5)
- moved R25 2.00 mm to (249.1, 107.0)
- moved R13 2.00 mm to (168.1, 100.5)
- moved R18 2.00 mm to (189.1, 107.0)
- moved R2 1.64 mm to (198.0, 81.0)
- moved R20 1.57 mm to (229.5, 100.0)
- moved R17 1.50 mm to (168.1, 107.0)
- moved R19 1.50 mm to (208.9, 107.0)
- moved R24 1.50 mm to (229.1, 107.0)
- moved R40 0.55 mm to (188.4, 251.5)
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Connections:
- A1 pad 1: /Button1 -> /Button14
- A1 pad 10: /Button8 -> /Button10
- A1 pad 11: /Button9 -> /Button20
- A1 pad 12: /Button10 -> /Button15
- A1 pad 14: /Button11 -> /Button8
- A1 pad 15: /Button12 -> /Button3
- A1 pad 16: /Button13 -> /Button17
- A1 pad 17: /Button14 -> /Button12
- A1 pad 19: /Button15 -> /Button7
- A1 pad 2: /Button2 -> /Button9
- A1 pad 20: /Button16 -> /Button1
- A1 pad 21: /Button17 -> Switch Pos 1
- A1 pad 22: /Button18 -> Switch Pos 2
- A1 pad 24: /Button19 -> Switch Pos 3
- A1 pad 25: /Button20 -> /Button6
- A1 pad 26: Switch Pos 1 -> /Button11
- A1 pad 27: Switch Pos 2 -> /Button16
- A1 pad 29: Switch Pos 3 -> /Button2
- A1 pad 4: /Button3 -> /Button4
- A1 pad 5: /Button4 -> /Button18
- A1 pad 6: /Button5 -> /Button13
- A1 pad 7: /Button6 -> /Button19
- A1 pad 9: /Button7 -> /Button5
Routing:
- net /Button18: track 15.9 -> 89.0 mm
- net Net-(S13-A): track 76.7 -> 8.23 mm
- net /Button13: track 15.4 -> 68.7 mm
- net Net-(S12-A): track 58.0 -> 7.78 mm
- net GND: track 0.00 -> 41.9 mm
- net +5V: track 758.3 -> 722.5 mm
- net +3.3V: track 0.00 -> 32.6 mm, vias 0 -> 4
- net /Button16: track 217.4 -> 237.9 mm
- net /Button2: track 251.4 -> 265.2 mm
- net Switch Pos 1: track 54.7 -> 40.9 mm
- net Potentiometer 2: track 229.1 -> 221.1 mm
- net Switch Pos 2: track 57.7 -> 50.0 mm
- net Net-(S5-A): track 0.00 -> 7.67 mm
- net /Button6: track 197.7 -> 190.3 mm
- net Switch Pos 3: track 62.7 -> 58.2 mm
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
Commit message: Update silkscreen
Other:
- board text added: "Raspberry Pi Pico 2"
- board text added: "Standalone F18 DDI v1.0 Tolga Cavusoglu December 2025"
Changed lines of the file:
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@@
 		(layer "Edge.Cuts")
+	)
+	(gr_text "Standalone F18 DDI v1.0\nTolga Cavusoglu\nDecember 2025"
+		(at 154 72.75 -0)
+		(layer "F.SilkS")
+		(effects
+			(font
+				(size 1 1)
+				(thickness 0.1)
+			)
+			(justify left bottom mirror)
+		)
+	)
+	(gr_text "Raspberry Pi Pico 2\n"
+		(at 277.5 97.75 0)
+		(layer "B.SilkS")
+		(effects
+			(font
+				(size 1 1)
+				(thickness 0.1)
+			)
+			(justify left bottom mirror)
+		)
 	)
 	(segment
